Commit message: Added final coordinate frame for end effector to URDF

File: src/planar_2d_description/urdf/planar_2d.urdf (robot description, URDF)
Before this commit: robot planar_2d, 3 links, 2 joints
Links:
- added link link3
Joints:
- added joint end_effector: type fixed, parent link2, child link3, origin xyz=.1 0 0 rpy=0 0 0, axis 0 0 1

Commit message: Finalized design in urdf. Used moveit setup assistant to configure robot arm.

File: src/planar_2d_description/urdf/planar_2d.urdf (robot description, URDF)
Before this commit: robot planar_2d, 4 links, 3 joints
Links:
- link link1: geometry visual cylinder length=0.127127 radius=.01905
- link link2: geometry visual cylinder length=0.146685 radius=0.01905
Joints:
- joint end_effector: origin xyz=.1 0 0 rpy=0 0 0 -> xyz=0.146685 0 0 rpy=0 0 0
- joint joint2: origin xyz=.1 0 0 rpy=0 0 0 -> xyz=0.127127 0 0 rpy=0 0 0
